File: torn_left/torn_left.sch (KiCad schematic (older format))
At the start: 76 parts, among them J1 SJ-43514, SW1 SW_Push, SW10 SW_Push, SW11 SW_Push, SW12 SW_Push, SW13 SW_Push, SW14 SW_Push, SW15 SW_Push, SW16 SW_Push, SW17 SW_Push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

Commit message: switched out SJ-43514 TRRS jack connector for PJ-320A
Parts:
- J1: footprint footprints:CUI_SJ-43514 -> footprints:PJ-320A; symbol SJ-43514:SJ-43514 -> torn_left-rescue:SJ-43514-SJ-43514
- USB1: symbol usb_c_gct_usb4085-type-c:USB_C_GCT_USB4085-Type-C -> torn_left-rescue:USB_C_GCT_USB4085-Type-C-usb_c_gct_usb4085-type-c
Changed lines of the file:
@@
 	3550 2250 3300 2250
 $Comp
-L usb_c_gct_usb4085-type-c:USB_C_GCT_USB4085-Type-C USB1
+L torn_left-rescue:USB_C_GCT_USB4085-Type-C-usb_c_gct_usb4085-type-c USB1
 U 1 1 5F4F038F
 P 2000 2300
@@
 $EndComp
 $Comp
-L SJ-43514:SJ-43514 J1
+L torn_left-rescue:SJ-43514-SJ-43514 J1
 U 1 1 5F2502D0
 P 5100 1950
 F 0 "J1" H 5157 2417 50  0000 C CNN
 F 1 "SJ-43514" H 5157 2326 50  0000 C CNN
-F 2 "footprints:CUI_SJ-43514" H 5100 1950 50  0001 L BNN
+F 2 "footprints:PJ-320A" H 5100 1950 50  0001 L BNN
 F 3 "1.04" H 5100 1950 50  0001 L BNN
 F 4 "MANUFACTURER RECOMMENDATIONS" H 5100 1950 50  0001 L BNN "Field4"
@@
 ENC0_A
 $Comp
-L power:GND #PWR?
+L power:GND #PWR0106
 U 1 1 5F73D838
 P 10450 900
-F 0 "#PWR?" H 10450 650 50  0001 C CNN
+F 0 "#PWR0106" H 10450 650 50  0001 C CNN
 F 1 "GND" H 10455 727 50  0000 C CNN
 F 2 "" H 10450 900 50  0001 C CNN
