File: torn_right/torn_right.sch (KiCad schematic (older format))
At the start: 64 parts, among them J2 SJ-43514, J3 Conn_01x04, SW23 SW_Push, SW24 SW_Push, SW25 SW_Push, SW26 SW_Push, SW27 SW_Push, SW28 Rotary_Encoder_Switch, SW29 SW_Push, SW30 SW_Push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

Commit message: switched out SJ-43514 TRRS jack connector for PJ-320A
Parts:
- J2: footprint footprints:CUI_SJ-43514 -> footprints:PJ-320A; symbol SJ-43514:SJ-43514 -> torn_right-rescue:SJ-43514-SJ-43514
Changed lines of the file:
@@
 	4350 4400 4350 4150
 $Comp
-L SJ-43514:SJ-43514 J2
+L torn_right-rescue:SJ-43514-SJ-43514 J2
 U 1 1 5F0C0BDE
 P 3650 4500
 F 0 "J2" H 3707 4967 50  0000 C CNN
 F 1 "SJ-43514" H 3707 4876 50  0000 C CNN
-F 2 "footprints:CUI_SJ-43514" H 3650 4500 50  0001 L BNN
+F 2 "footprints:PJ-320A" H 3650 4500 50  0001 L BNN
 F 3 "1.04" H 3650 4500 50  0001 L BNN
 F 4 "MANUFACTURER RECOMMENDATIONS" H 3650 4500 50  0001 L BNN "Field4"
